Commit message: update prject

File: src/my_robot/urdf/my_robot.xacro (robot description, xacro)
@@ -165,4 +165,7 @@
   <link name="camera_link_optical">
   </link>
+  <gazebo reference="camera">
+      <material>Gazebo/White</material>
+  </gazebo>
   <!-- HOKUYO LIDAR -->
   <joint type="fixed" name="hukoyo_joint">
